File: ac-dc-converter-mp171.sch (KiCad schematic (older format))
At the start: 18 parts, among them J1 Conn_01x01, J2 Conn_01x01, J3 Conn_01x05, U1 MP171GJ

Commit message: completed so far. ready to order.
Parts:
- removed J3: Conn_01x05, Connector_PinHeader_2.54mm:PinHeader_1x05_P2.54mm_Vertical, symbol Connector_Generic:Conn_01x05
- added C1: 1u_400V, Capacitor_THT:CP_Radial_D6.3mm_P2.50mm, symbol _C_Electrolytic:1u_400V
- added D4: LED, LED_SMD:LED_0603_1608Metric, symbol Device:LED
- added J3, J4: Conn_01x01, Connector_PinHeader_2.54mm:PinHeader_1x01_P2.54mm_Vertical, symbol Connector_Generic:Conn_01x01
- added L1: 330uH, Inductor_SMD:L_1210_3225Metric, symbol _L_1210:330uH
- added R3: 1K, Resistor_SMD:R_0603_1608Metric, symbol _R_0603:1K
- renumbered C1 to C2, C2 to C3, C3 to C4, C4 to C5, C5 to C6, C6 to C7, L1 to L2, L2 to L3, L3 to L4
Connections:
- net +5V1: now also J3.1 (Pin_1), R3.1
- net DRAIN: now also L1.2; no longer D1.1 (K)
- net GND: now also C1.2, D4.1 (K), J4.1 (Pin_1)
- new net: C1.1, D1.1 (K), L1.1
- new net: D4.2 (A), R3.2
Other:
- moved on the sheet: D1, J1, J2
